Commit message: 修复事件管理器类实例化问题并更新Taks T1机器人URDF惯性参数
- 事件管理器中添加类实例化检查,确保基于类的事件项在调用前正确初始化
- 为randomize_rigid_body_inertia和randomize_joint_parameters事件添加默认参数值
- 修复randomize_joint_parameters中armature写入时的索引错误,正确处理slice类型的joint_ids
- 更新Taks T1机器人URDF文件中所有关节的惯性参数(质量、质心位置、惯性张量)和关节原点坐标,

File: source/isaaclab_assets/isaaclab_assets/robots/Taks_T1/Taks_T1.urdf (robot description, URDF)
Before this commit: robot Taks_T1, 33 links, 32 joints
Links:
- link left_ankle_pitch_link: mass 0.001837 -> 0.23
- link left_ankle_roll_link: mass 0.56 -> 0.15
- link left_hip_pitch_link: mass 0.685 -> 0.91
- link left_hip_roll_link: mass 0.93 -> 0.79
- link left_hip_yaw_link: mass 1.74 -> 1.822
- link left_knee_link: mass 0.63 -> 1.138
- link pelvis: mass 3.2 -> 3.34
- link right_ankle_pitch_link: mass 0.001837 -> 0.23
- link right_ankle_roll_link: mass 0.56 -> 0.15
- link right_hip_pitch_link: mass 0.685 -> 0.91
- link right_hip_roll_link: mass 0.93 -> 0.79
- link right_hip_yaw_link: mass 1.74 -> 1.822
- link right_knee_link: mass 0.63 -> 1.138
Joints:
- joint left_ankle_pitch_joint: origin xyz=0.0 -0.015197 -0.28503 rpy=0 0 0 -> xyz=0.0 0.0227 -0.2985 rpy=0 0 0
- joint left_ankle_roll_joint: origin xyz=0.02 0.0 0.0 rpy=0 0 0 -> xyz=0.04 -0.024 0.0 rpy=0 0 0
- joint left_hip_pitch_joint: origin xyz=0.0 0.115 -0.0523 rpy=0 0 0 -> xyz=0.0 0.0919 -0.08747 rpy=0 0 0
- joint left_hip_roll_joint: origin xyz=0.007945 0.053348 0.001351 rpy=0.0 -0.1745333851200459 0.0 -> xyz=0.00795 0.0765 -0.04167 rpy=0.0 -0.17453 0.0
- joint left_hip_yaw_joint: origin xyz=-0.008293 0.0 -0.10937 rpy=0 0 0 -> xyz=0.00829 0.0 -0.1094 rpy=0 0 0
- joint left_knee_joint: origin xyz=-0.060138 0.016849 -0.23297 rpy=0.0 0.17453338512004613 0.0 -> xyz=-0.0484 0.0 -0.1665 rpy=0.0 0.17453 0.0
- joint right_ankle_pitch_joint: origin xyz=0.0 0.015197 -0.28503 rpy=0 0 0 -> xyz=0.0 -0.0222 -0.2985 rpy=0 0 0
- joint right_ankle_roll_joint: origin xyz=0.02 0.0 0.0 rpy=0 0 0 -> xyz=0.04 0.024 0.0 rpy=0 0 0
- joint right_hip_pitch_joint: origin xyz=0.0 -0.115 -0.0523 rpy=0 0 0 -> xyz=0.0 -0.0913 -0.08747 rpy=0 0 0
- joint right_hip_roll_joint: origin xyz=0.007945 -0.053348 0.001351 rpy=0.0 -0.1745333851200459 0.0 -> xyz=0.00795 -0.077 -0.04167 rpy=0.0 -0.17453 0.0
- joint right_hip_yaw_joint: origin xyz=-0.008293 0.0 -0.10937 rpy=0 0 0 -> xyz=0.00829 0.0 -0.1094 rpy=0 0 0
- joint right_knee_joint: origin xyz=-0.060138 -0.016849 -0.23297 rpy=0.0 0.17453338512004613 0.0 -> xyz=-0.0484 -0.0005 -0.1665 rpy=0.0 0.17453 0.0

Commit message: 优化Taks T1机器人脚部碰撞几何和手臂关节默认位置:将脚踝碰撞从网格模型替换为四点球体布局,调整手腕惯性参数,并优化肩部和肘部关节初始角度
- 左右脚踝碰撞几何从单一网格模型替换为四个半径0.005的球体,分布于脚底四角(-0.08/0.08, ±0.025, -0.05)
- 左右手腕惯性参数更新:质量从0.28增至0.308,质心位置和转动惯量矩阵相应调整
- 肩部俯仰关节默认位置从0.17调整至0.20
- 肘部关节默

File: source/isaaclab_assets/isaaclab_assets/robots/Taks_T1/Taks_T1.urdf (robot description, URDF)
Before this commit: robot Taks_T1, 33 links, 32 joints
Links:
- link left_ankle_roll_link: geometry collision sphere radius=0.005; collision sphere radius=0.005
- link left_wrist_pitch_link: mass 0.28 -> 0.308
- link right_ankle_roll_link: geometry collision sphere radius=0.005; collision sphere radius=0.005
- link right_wrist_pitch_link: mass 0.28 -> 0.308

Commit message: 限制Taks T1机器人颈部关节活动范围并降低颈部偏差惩罚权重:将颈部yaw/roll/pitch三关节活动范围从±1.57/±0.873弧度严格限制至±0.001弧度以固定头部姿态,同时将颈部关节偏差惩罚权重从-0.2降至-0.1,并缩短Flat环境训练迭代次数从1100至501
- URDF和USD文件中颈部三关节(neck_yaw/roll/pitch)活动范围从原有范围限制至±0.001弧度
- Rough环境(含backup版本)颈部关节偏差惩罚权重从-0.2降至-0.1
- Flat环境max

File: source/isaaclab_assets/isaaclab_assets/robots/Taks_T1/Taks_T1.urdf (robot description, URDF)
Before this commit: robot Taks_T1, 33 links, 32 joints
Joints:
- joint neck_pitch_joint: limit lower=-0.873 upper=0.873 effort=3.0 velocity=15.71 -> lower=-0.001 upper=0.001 effort=3.0 velocity=15.71
- joint neck_roll_joint: limit lower=-0.873 upper=0.873 effort=3.0 velocity=15.71 -> lower=-0.001 upper=0.001 effort=3.0 velocity=15.71
- joint neck_yaw_joint: limit lower=-1.57 upper=1.57 effort=3.0 velocity=15.71 -> lower=-0.001 upper=0.001 effort=3.0 velocity=15.71
